File: custom_pcbs/breakout_board/breakout_board.kicad_pcb (KiCad board)
At the start: 4 copper layers, 30 x 65 mm, 6 parts, among them J1 INPUT_FROM_PI, J2 PMW3901_OUT

Commit message: Added more sensors
Parts:
- added VL53L1X_1_OUT: Conn_01x06, Connector_PinHeader_2.54mm:PinHeader_1x06_P2.54mm_Vertical, F.Cu at (138.0, 36.0)
- added VL53L1X_2_OUT: Conn_01x06, Connector_PinHeader_2.54mm:PinHeader_1x06_P2.54mm_Vertical, F.Cu at (138.0, 27.0)
- moved J2 10.4 mm to (156.0, 50.3)
- moved J1 7.96 mm to (133.9, 48.0)
Connections:
- J1 pad 10: unconnected-(J1-Pin_10-Pad10) -> /XSHUT_2
- J1 pad 7: unconnected-(J1-Pin_7-Pad7) -> /I2C_SDA
- J1 pad 8: unconnected-(J1-Pin_8-Pad8) -> /I2C_SCL
- J1 pad 9: unconnected-(J1-Pin_9-Pad9) -> /XSHUT_1
Routing:
- net /XSHUT_2: track 0.00 -> 58.3 mm
- net /I2C_SCL: track 0.00 -> 43.6 mm
- net /I2C_SDA: track 0.00 -> 40.0 mm
- net /XSHUT_1: track 0.00 -> 39.2 mm
- net +3V3: track 22.0 -> 45.8 mm
- net /SPI_MOSI: track 22.0 -> 23.2 mm
- net /SPI_CS: track 22.0 -> 23.2 mm
- net /SPI_MISO: track 23.0 -> 24.1 mm
- net /SPI_CLK: track 23.1 -> 24.0 mm, vias 0 -> 2
Other:
- board text removed: "JLCJLCJLCJLC"
