File: custom_pcbs/breakout_board/breakout_board.kicad_pcb (KiCad board)
At the start: 4 copper layers, 30 x 65 mm, 8 parts, among them J1 INPUT_FROM_PI, J2 PMW3901_OUT

Commit message: break out board design
Other:
- board text added: "INT"
- board text added: "Pin 11"
- board text added: "Pin 13"
- board text added: "Pin 3"
- board text added: "Pin 5"
- board text added: "SCL"
- board text added: "SDA"
- board text added: "SHUT"
- board text added: "VIN"
